File: doc/hw_filter/PLP-200+.brd (EAGLE design)
At the start: 27.9 x 30 mm, 3 parts

Commit message: updated libraries
Parts:
- LPF: device rct_lpf_brd:A01 -> PLP-200+:A01
- moved SMA_IN 22.9 mm to (6.35, 3.56), turned to 180 degrees
- moved SMA_OUT 22.9 mm to (21.6, 26.4), turned to 0 degrees
Changed lines of the file:
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@@
 </autorouter>
 <elements>
-<element name="LPF" library="rct_lpf_brd" package="A01" value="PLP-200+" x="13.97" y="14.986"/>
-<element name="SMA_IN" library="balun" package="SMA_EDGE_MNT" value="CONSMA013.062_JACKEND_MNT" x="6.35" y="26.416"/>
-<element name="SMA_OUT" library="balun" package="SMA_EDGE_MNT" value="CONSMA013.062END_MNT" x="21.59" y="3.556" rot="R180"/>
+<element name="LPF" library="PLP-200+" package="A01" value="PLP-200+" x="13.97" y="14.986"/>
+<element name="SMA_IN" library="balun" package="SMA_EDGE_MNT" value="CONSMA013.062_JACKEND_MNT" x="6.35" y="3.556" rot="R180"/>
+<element name="SMA_OUT" library="balun" package="SMA_EDGE_MNT" value="CONSMA013.062END_MNT" x="21.59" y="26.416"/>
 </elements>
 <signals>
@@
 <contactref element="SMA_IN" pad="SIG"/>
 <contactref element="LPF" pad="P1"/>
-<wire x1="6.35" y1="26.416" x2="6.35" y2="17.526" width="1.6256" layer="1"/>
+<wire x1="6.35" y1="3.556" x2="6.35" y2="12.446" width="1.6764" layer="1"/>
 </signal>
 <signal name="N$2">
 <contactref element="LPF" pad="P8"/>
 <contactref element="SMA_OUT" pad="SIG"/>
-<wire x1="21.59" y1="3.556" x2="21.59" y2="12.446" width="1.6256" layer="1"/>
+<wire x1="21.59" y1="26.416" x2="21.59" y2="17.526" width="1.6764" layer="1"/>
 </signal>
 <signal name="GND">
-<polygon width="0.4064" layer="1">
+<polygon width="0.4064" layer="1" isolate="0.254">
 <vertex x="1.27" y="28.702"/>
 <vertex x="26.67" y="28.702"/>
@@
 <vertex x="1.27" y="1.27"/>
 </polygon>
-<polygon width="0.4064" layer="16">
+<polygon width="0.4064" layer="16" isolate="0.254">
 <vertex x="1.27" y="28.702"/>
 <vertex x="26.67" y="28.702"/>
@@
 <via x="2.54" y="17.78" extent="1-16" drill="0.8"/>
 <via x="2.54" y="15.24" extent="1-16" drill="0.8"/>
-<via x="2.54" y="2.54" extent="1-16" drill="0.8"/>
-<via x="5.08" y="2.54" extent="1-16" drill="0.8"/>
-<via x="7.62" y="2.54" extent="1-16" drill="0.8"/>
-<via x="10.16" y="2.54" extent="1-16" drill="0.8"/>
+<via x="2.54" y="25.4" extent="1-16" drill="0.8"/>
+<via x="5.08" y="27.94" extent="1-16" drill="0.8"/>
+<via x="7.62" y="27.94" extent="1-16" drill="0.8"/>
+<via x="10.16" y="25.4" extent="1-16" drill="0.8"/>
 <via x="12.7" y="2.54" extent="1-16" drill="0.8"/>
 <via x="15.24" y="2.54" extent="1-16" drill="0.8"/>
-<via x="2.54" y="5.08" extent="1-16" drill="0.8"/>
-<via x="5.08" y="5.08" extent="1-16" drill="0.8"/>
-<via x="7.62" y="5.08" extent="1-16" drill="0.8"/>
-<via x="10.16" y="5.08" extent="1-16" drill="0.8"/>
+<via x="2.54" y="27.94" extent="1-16" drill="0.8"/>
+<via x="5.08" y="25.4" extent="1-16" drill="0.8"/>
+<via x="7.62" y="25.4" extent="1-16" drill="0.8"/>
+<via x="10.16" y="27.94" extent="1-16" drill="0.8"/>
 <via x="12.7" y="5.08" extent="1-16" drill="0.8"/>
 <via x="15.24" y="5.08" extent="1-16" drill="0.8"/>
 <via x="2.54" y="7.62" extent="1-16" drill="0.8"/>
-<via x="5.08" y="7.62" extent="1-16" drill="0.8"/>
-<via x="7.62" y="7.62" extent="1-16" drill="0.8"/>
+<via x="5.08" y="22.86" extent="1-16" drill="0.8"/>
+<via x="7.62" y="22.86" extent="1-16" drill="0.8"/>
 <via x="10.16" y="7.62" extent="1-16" drill="0.8"/>
 <via x="12.7" y="7.62" extent="1-16" drill="0.8"/>
@@
 <via x="2.54" y="10.16" extent="1-16" drill="0.8"/>
 <via x="2.54" y="12.7" extent="1-16" drill="0.8"/>
-<via x="5.08" y="10.16" extent="1-16" drill="0.8"/>
-<via x="7.62" y="10.16" extent="1-16" drill="0.8"/>
+<via x="5.08" y="20.32" extent="1-16" drill="0.8"/>
+<via x="7.62" y="20.32" extent="1-16" drill="0.8"/>
 <via x="10.16" y="10.16" extent="1-16" drill="0.8"/>
 <via x="12.7" y="10.16" extent="1-16" drill="0.8"/>
@@
 <via x="25.4" y="17.78" extent="1-16" drill="0.8"/>
 <via x="25.4" y="20.32" extent="1-16" drill="0.8"/>
-<via x="22.86" y="20.32" extent="1-16" drill="0.8"/>
-<via x="20.32" y="20.32" extent="1-16" drill="0.8"/>
+<via x="22.86" y="2.54" extent="1-16" drill="0.8"/>
+<via x="20.32" y="2.54" extent="1-16" drill="0.8"/>
 <via x="17.78" y="20.32" extent="1-16" drill="0.8"/>
 <via x="15.24" y="20.32" extent="1-16" drill="0.8"/>
@@
 <via x="15.24" y="22.86" extent="1-16" drill="0.8"/>
 <via x="17.78" y="22.86" extent="1-16" drill="0.8"/>
-<via x="17.78" y="25.4" extent="1-16" drill="0.8"/>
-<via x="17.78" y="27.94" extent="1-16" drill="0.8"/>
-<via x="20.32" y="25.4" extent="1-16" drill="0.8"/>
-<via x="20.32" y="27.94" extent="1-16" drill="0.8"/>
-<via x="20.32" y="22.86" extent="1-16" drill="0.8"/>
-<via x="22.86" y="22.86" extent="1-16" drill="0.8"/>
-<via x="22.86" y="25.4" extent="1-16" drill="0.8"/>
-<via x="22.86" y="27.94" extent="1-16" drill="0.8"/>
-<via x="25.4" y="27.94" extent="1-16" drill="0.8"/>
-<via x="25.4" y="25.4" extent="1-16" drill="0.8"/>
+<via x="17.78" y="5.08" extent="1-16" drill="0.8"/>
+<via x="17.78" y="2.54" extent="1-16" drill="0.8"/>
+<via x="20.32" y="7.62" extent="1-16" drill="0.8"/>
+<via x="20.32" y="10.16" extent="1-16" drill="0.8"/>
+<via x="20.32" y="5.08" extent="1-16" drill="0.8"/>
+<via x="22.86" y="5.08" extent="1-16" drill="0.8"/>
+<via x="22.86" y="7.62" extent="1-16" drill="0.8"/>
+<via x="22.86" y="10.16" extent="1-16" drill="0.8"/>
+<via x="25.4" y="5.08" extent="1-16" drill="0.8"/>
+<via x="25.4" y="2.54" extent="1-16" drill="0.8"/>
 <via x="25.4" y="22.86" extent="1-16" drill="0.8"/>
 </signal>
