File: doc/hw_filter/sxbp-169.brd (EAGLE design)
At the start: 25.4 x 40.6 mm, 3 parts

Commit message: updated libraries
Connections:
- net RF_IN renamed N$1
- net RF_OUT renamed N$3
Routing:
- net GND: track 47.6 -> 0.00 mm, vias 24 -> 20
Changed lines of the file:
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@@
 <?xml version="1.0" encoding="utf-8"?>
 <!DOCTYPE eagle SYSTEM "eagle.dtd">
-<eagle version="7.2.0">
+<eagle version="8.0.0">
 <drawing>
 <settings>
@@
 <layers>
 <layer number="1" name="Top" color="4" fill="1" visible="yes" active="yes"/>
+<layer number="2" name="Route2" color="1" fill="3" visible="no" active="no"/>
+<layer number="3" name="Route3" color="4" fill="3" visible="no" active="no"/>
+<layer number="4" name="Route4" color="1" fill="4" visible="no" active="no"/>
+<layer number="5" name="Route5" color="4" fill="4" visible="no" active="no"/>
+<layer number="6" name="Route6" color="1" fill="8" visible="no" active="no"/>
+<layer number="7" name="Route7" color="4" fill="8" visible="no" active="no"/>
+<layer number="8" name="Route8" color="1" fill="2" visible="no" active="no"/>
+<layer number="9" name="Route9" color="4" fill="2" visible="no" active="no"/>
+<layer number="10" name="Route10" color="1" fill="7" visible="no" active="no"/>
+<layer number="11" name="Route11" color="4" fill="7" visible="no" active="no"/>
+<layer number="12" name="Route12" color="1" fill="5" visible="no" active="no"/>
+<layer number="13" name="Route13" color="4" fill="5" visible="no" active="no"/>
+<layer number="14" name="Route14" color="1" fill="6" visible="no" active="no"/>
+<layer number="15" name="Route15" color="4" fill="6" visible="no" active="no"/>
 <layer number="16" name="Bottom" color="1" fill="1" visible="yes" active="yes"/>
 <layer number="17" name="Pads" color="2" fill="1" visible="yes" active="yes"/>
@@
 </autorouter>
 <elements>
-<element name="FILTER" library="balun" package="HF1139" value="SXBP-169+SXBP-169+" x="12.7" y="20.32"/>
 <element name="INPUT" library="balun" package="SMA_EDGE_MNT" value="CONSMA013.062_JACKEND_MNT" x="12.7" y="2.921" rot="R180"/>
 <element name="OUTPUT" library="balun" package="SMA_EDGE_MNT" value="CONSMA013.062END_MNT" x="12.7" y="37.719"/>
+<element name="FILTER" library="balun" package="HF1139" value="SXBP-169+SXBP-169+" x="12.7" y="20.32"/>
 </elements>
 <signals>
-<signal name="RF_IN">
-<contactref element="INPUT" pad="SIG"/>
-<contactref element="FILTER" pad="RF_IN"/>
-<wire x1="12.7" y1="2.921" x2="12.7" y2="6.35" width="1.6256" layer="1"/>
-<wire x1="12.7" y1="6.35" x2="5.08" y2="13.97" width="1.6256" layer="1"/>
-<wire x1="5.08" y1="13.97" x2="5.08" y2="15.0495" width="1.6256" layer="1"/>
-</signal>
-<signal name="RF_OUT">
-<contactref element="OUTPUT" pad="SIG"/>
-<contactref element="FILTER" pad="RF_OUT"/>
-<wire x1="12.7" y1="37.719" x2="12.7" y2="34.29" width="1.6256" layer="1"/>
-<wire x1="12.7" y1="34.29" x2="20.32" y2="26.67" width="1.6256" layer="1"/>
-<wire x1="20.32" y1="26.67" x2="20.32" y2="25.5905" width="1.6256" layer="1"/>
-</signal>
 <signal name="GND">
-<polygon width="0.3048" layer="1">
-<vertex x="8.89" y="13.97"/>
-<vertex x="8.89" y="19.5072"/>
-<vertex x="3.81" y="19.5072"/>
-<vertex x="3.81" y="26.67"/>
-<vertex x="16.51" y="26.67"/>
-<vertex x="16.51" y="21.1328"/>
-<vertex x="21.59" y="21.1328"/>
-<vertex x="21.59" y="13.97"/>
-</polygon>
-<polygon width="0.3048" layer="16">
+<polygon width="0.3048" layer="16" isolate="0.254">
 <vertex x="1.27" y="39.37"/>
 <vertex x="1.27" y="1.27"/>
 <vertex x="7.62" y="1.27"/>
-<vertex x="7.62" y="6.35"/>
-<vertex x="17.78" y="6.35"/>
 <vertex x="17.78" y="1.27"/>
 <vertex x="24.13" y="1.27"/>
 <vertex x="24.13" y="39.37"/>
 <vertex x="17.78" y="39.37"/>
-<vertex x="17.78" y="34.29"/>
-<vertex x="7.62" y="34.29"/>
 <vertex x="7.62" y="39.37"/>
 </polygon>
-<contactref element="INPUT" pad="GND1"/>
-<contactref element="INPUT" pad="GND2"/>
-<contactref element="FILTER" pad="GND3"/>
-<contactref element="FILTER" pad="GND5"/>
-<contactref element="FILTER" pad="GND7"/>
-<contactref element="FILTER" pad="GND6"/>
-<contactref element="FILTER" pad="GND2"/>
-<contactref element="FILTER" pad="GND4"/>
-<contactref element="OUTPUT" pad="GND2"/>
-<contactref element="OUTPUT" pad="GND1"/>
-<contactref element="INPUT" pad="GND3"/>
-<contactref element="INPUT" pad="GND4"/>
-<contactref element="OUTPUT" pad="GND3"/>
-<contactref element="OUTPUT" pad="GND4"/>
-<wire x1="10.16" y1="37.719" x2="10.16" y2="33.02" width="1.6256" layer="16"/>
-<wire x1="15.24" y1="37.719" x2="15.24" y2="33.02" width="1.6256" layer="16"/>
-<wire x1="10.16" y1="2.921" x2="10.16" y2="6.35" width="1.6256" layer="16"/>
-<wire x1="15.24" y1="2.921" x2="15.24" y2="6.35" width="1.6256" layer="16"/>
 <via x="2.54" y="38.1" extent="1-16" drill="0.6"/>
 <via x="2.54" y="34.29" extent="1-16" drill="0.6"/>
 <via x="2.54" y="30.48" extent="1-16" drill="0.6"/>
 <via x="6.35" y="30.48" extent="1-16" drill="0.6"/>
-<via x="6.35" y="34.29" extent="1-16" drill="0.6"/>
 <via x="6.35" y="38.1" extent="1-16" drill="0.6"/>
 <via x="10.16" y="30.48" extent="1-16" drill="0.6"/>
-<via x="19.05" y="34.29" extent="1-16" drill="0.6"/>
 <via x="19.05" y="38.1" extent="1-16" drill="0.6"/>
 <via x="22.86" y="38.1" extent="1-16" drill="0.6"/>
@@
 <via x="2.54" y="2.54" extent="1-16" drill="0.6"/>
 <via x="6.35" y="2.54" extent="1-16" drill="0.6"/>
-<via x="6.35" y="6.35" extent="1-16" drill="0.6"/>
 <via x="15.24" y="10.16" extent="1-16" drill="0.6"/>
 <via x="19.05" y="10.16" extent="1-16" drill="0.6"/>
-<via x="19.05" y="6.35" extent="1-16" drill="0.6"/>
 <via x="19.05" y="2.54" extent="1-16" drill="0.6"/>
 <via x="22.86" y="2.54" extent="1-16" drill="0.6"/>
 <via x="22.86" y="6.35" extent="1-16" drill="0.6"/>
 <via x="22.86" y="10.16" extent="1-16" drill="0.6"/>
-<polygon width="0.3048" layer="1">
+<polygon width="0.4064" layer="1" isolate="0.254">
+<vertex x="1.27" y="39.37"/>
+<vertex x="24.13" y="39.37"/>
+<vertex x="24.13" y="1.27"/>
 <vertex x="1.27" y="1.27"/>
-<vertex x="7.62" y="1.27"/>
-<vertex x="7.62" y="6.35"/>
-<vertex x="10.16" y="6.35"/>
-<vertex x="2.54" y="13.97"/>
-<vertex x="1.27" y="13.97"/>
 </polygon>
-<polygon width="0.3048" layer="1">
-<vertex x="15.24" y="6.35"/>
-<vertex x="8.89" y="12.7"/>
-<vertex x="24.13" y="12.7"/>
-<vertex x="24.13" y="1.27"/>
-<vertex x="17.78" y="1.27"/>
-<vertex x="17.78" y="6.35"/>
-</polygon>
-<polygon width="0.3048" layer="1">
-<vertex x="1.27" y="39.37"/>
-<vertex x="7.62" y="39.37"/>
-<vertex x="7.62" y="34.29"/>
-<vertex x="10.16" y="34.29"/>
-<vertex x="16.51" y="27.94"/>
-<vertex x="1.27" y="27.94"/>
-</polygon>
-<polygon width="0.3048" layer="1">
-<vertex x="17.78" y="39.37"/>
-<vertex x="17.78" y="34.29"/>
-<vertex x="15.24" y="34.29"/>
-<vertex x="22.86" y="26.67"/>
-<vertex x="24.13" y="26.67"/>
-<vertex x="24.13" y="39.37"/>
-</polygon>
-<wire x1="15.24" y1="15.0495" x2="15.24" y2="12.7" width="1.6256" layer="1"/>
-<wire x1="10.16" y1="2.921" x2="6.35" y2="2.921" width="1.6256" layer="1"/>
-<wire x1="6.35" y1="2.921" x2="6.35" y2="6.35" width="1.6256" layer="1"/>
-<wire x1="15.24" y1="2.921" x2="19.05" y2="2.921" width="1.6256" layer="1"/>
-<wire x1="19.05" y1="2.921" x2="19.05" y2="6.35" width="1.6256" layer="1"/>
-<wire x1="15.24" y1="37.719" x2="19.05" y2="37.719" width="1.6256" layer="1"/>
-<wire x1="19.05" y1="37.719" x2="19.05" y2="34.29" width="1.6256" layer="1"/>
-<wire x1="10.16" y1="37.719" x2="6.35" y2="37.719" width="1.6256" layer="1"/>
-<wire x1="6.35" y1="37.719" x2="6.35" y2="34.29" width="1.6256" layer="1"/>
+<contactref element="INPUT" pad="GND1"/>
+<contactref element="INPUT" pad="GND2"/>
+<contactref element="INPUT" pad="GND4"/>
+<contactref element="INPUT" pad="GND3"/>
+<contactref element="FILTER" pad="GND5"/>
+<contactref element="FILTER" pad="GND2"/>
+<contactref element="FILTER" pad="GND3"/>
+<contactref element="FILTER" pad="GND7"/>
+<contactref element="FILTER" pad="GND4"/>
+<contactref element="FILTER" pad="GND6"/>
+<contactref element="OUTPUT" pad="GND1"/>
+<contactref element="OUTPUT" pad="GND2"/>
+<contactref element="OUTPUT" pad="GND4"/>
+<contactref element="OUTPUT" pad="GND3"/>
+</signal>
+<signal name="N$1">
+<contactref element="INPUT" pad="SIG"/>
+<contactref element="FILTER" pad="RF_IN"/>
+<wire x1="12.7" y1="2.921" x2="12.7" y2="6.35" width="1.6764" layer="1"/>
+<wire x1="12.7" y1="6.35" x2="5.08" y2="13.97" width="1.6764" layer="1"/>
+<wire x1="5.08" y1="13.97" x2="5.08" y2="15.0495" width="1.6764" layer="1"/>
+</signal>
+<signal name="N$3">
+<contactref element="OUTPUT" pad="SIG"/>
+<contactref element="FILTER" pad="RF_OUT"/>
+<wire x1="12.7" y1="37.719" x2="12.7" y2="34.29" width="1.6764" layer="1"/>
+<wire x1="12.7" y1="34.29" x2="20.32" y2="26.67" width="1.6764" layer="1"/>
+<wire x1="20.32" y1="26.67" x2="20.32" y2="25.5905" width="1.6764" layer="1"/>
+</signal>
+<signal name="N$5">
 </signal>
 </signals>
